Commit message: safety walls

File: src/Universal_Robots_ROS2_Tutorials/my_robot_cell/my_robot_cell_description/urdf/my_robot_cell.urdf.xacro (robot description, xacro)
@@ -17,5 +17,5 @@
     visual_parameters_file="$(arg visual_parameters_file)"
     >
-      <origin xyz="0 0 1" rpy="0 0 0" />
+      <origin xyz="0 0 0" rpy="0 0 0" />
   </xacro:my_robot_cell>
 </robot>

File: src/Universal_Robots_ROS2_Tutorials/my_robot_cell/my_robot_cell_description/urdf/my_robot_cell_macro.xacro (robot description, xacro)
@@ -2,4 +2,6 @@
 <robot xmlns:xacro="http://ros.org/wiki/xacro">
   <xacro:include filename="$(find ur_description)/urdf/ur_macro.xacro"/>
+  <xacro:include filename="$(find my_robot_cell_description)/urdf/safety_wall.xacro"/>
+  <xacro:include filename="$(find my_robot_cell_description)/urdf/table.xacro"/>
   <xacro:macro name="my_robot_cell" params="
     parent
@@ -11,65 +13,15 @@
     visual_parameters_file
     ">
-    <joint name="table_base_joint" type="fixed">
-      <xacro:insert_block name="origin" />
-      <parent link="${parent}" />
-      <child link="table" />
-    </joint>
-    <link name="table">
-      <visual>
-        <geometry>
-          <mesh filename="package://my_robot_cell_description/meshes/fzi_table.dae"/>
-        </geometry>
-        <origin rpy="0 0 0" xyz="0.75 0.5 -1"/>
-      </visual>
-      <collision>
-        <geometry>
-          <mesh filename="package://my_robot_cell_description/meshes/fzi_table.dae"/>
-        </geometry>
-        <origin rpy="0 0 0" xyz="0.75 0.5 -1"/>
-      </collision>
-    </link>
-    <link name="monitor">
-      <visual>
-        <geometry>
-          <mesh filename="package://my_robot_cell_description/meshes/171005_Motek_Monitor_L.dae"/>
-        </geometry>
-      </visual>
-      <collision>
-        <geometry>
-          <mesh filename="package://my_robot_cell_description/meshes/171005_Motek_Monitor_L.dae"/>
-        </geometry>
-      </collision>
-    </link>
-    <joint name="base_to_monitor" type="fixed">
-      <parent link="table"/>
-      <child link="monitor"/>
-      <origin xyz="0.2 0.6 0"/>
-    </joint>
-    <material name="white">
-      <color rgba="1 1 1 1"/>
-    </material>
-    <link name="wall">
-      <visual>
-        <geometry>
-          <mesh filename="package://my_robot_cell_description/meshes/wall.dae"/>
-        </geometry>
-      </visual>
-      <collision>
-        <geometry>
-          <box size="4.44 0.1 2.5"/>
-        </geometry>
-      </collision>
-    </link>
-    <joint name="base_to_wall" type="fixed">
-      <parent link="table"/>
-      <child link="wall"/>
-      <origin xyz="1.25 1.5 0.5"/>
-    </joint>
+    <xacro:table parent="${parent}">
+      <origin rpy="0 0 0" xyz="0 -0 0.9"/>
+    </xacro:table>
+    <xacro:safety_wall parent="${parent}">
+      <origin rpy="0 0 0" xyz="0 0 0"/>
+    </xacro:safety_wall>
     <link name="robot_mount"/>
     <joint name="base_to_robot_mount" type="fixed">
-      <parent link="table"/>
+      <parent link="robot_base_plate"/>
       <child link="robot_mount"/>
-      <origin xyz="0.845 0.85 0" rpy="0 0 ${pi}" />
+      <origin xyz="0 0 0" rpy="0 0 ${pi}" />
     </joint>
     <!--This will create the specific robot-->
