Commit message: gipper

File: src/Universal_Robots_ROS2_Tutorials/my_robot_cell/my_robot_cell_description/urdf/my_robot_cell_macro.xacro (robot description, xacro)
@@ -4,4 +4,6 @@
   <xacro:include filename="$(find my_robot_cell_description)/urdf/safety_wall.xacro"/>
   <xacro:include filename="$(find my_robot_cell_description)/urdf/table.xacro"/>
+  <xacro:include filename="$(find my_robot_cell_description)/urdf/box.xacro"/>
+  <xacro:include filename="$(find my_robot_cell_description)/urdf/2fg7_gripper/urdf/onrobot_2fg7_gripper.urdf.xacro"/>
   <xacro:macro name="my_robot_cell" params="
     parent
@@ -37,4 +39,10 @@
       <origin xyz="0 0 0" rpy="0 0 0" />
     </xacro:ur_robot>
+    <xacro:box parent="ur5e_tool0">
+      <origin xyz="0 0 0.1" rpy="0 0 0"/>
+    </xacro:box>
+    <!--xacro:onrobot_2fg7_gripper prefix= "onrobot_2fg7_gripper" parent="ur5e_tool0">
+      <origin yxz="0 0 0" rpy="0 4.71239 0"/>
+    </xacro:onrobot_2fg7_gripper-->
   </xacro:macro>
 </robot>
