Commit message: defining one robot, ready to add second one in world

File: src/Universal_Robots_ROS2_Tutorials/my_robot_cell/moveit_config/config/my_robot_cell.ros2_control.xacro (robot description, xacro)
@@ -8,51 +8,63 @@
                 <plugin>mock_components/GenericSystem</plugin>
             </hardware>
-            <joint name="ur5e_shoulder_pan_joint">
+            <joint name="ur5e_409_shoulder_pan_joint">
                 <command_interface name="position"/>
                 <command_interface name="velocity"/>
+                <command_interface name="effort"/>
                 <state_interface name="position">
-                  <param name="initial_value">${initial_positions['ur5e_shoulder_pan_joint']}</param>
+                  <param name="initial_value">${initial_positions['ur5e_409_shoulder_pan_joint']}</param>
                 </state_interface>
                 <state_interface name="velocity"/>
+                <state_interface name="effort"/>
             </joint>
-            <joint name="ur5e_shoulder_lift_joint">
+            <joint name="ur5e_409_shoulder_lift_joint">
                 <command_interface name="position"/>
                 <command_interface name="velocity"/>
+                <command_interface name="effort"/>
                 <state_interface name="position">
-                  <param name="initial_value">${initial_positions['ur5e_shoulder_lift_joint']}</param>
+                  <param name="initial_value">${initial_positions['ur5e_409_shoulder_lift_joint']}</param>
                 </state_interface>
                 <state_interface name="velocity"/>
+                <state_interface name="effort"/>
             </joint>
-            <joint name="ur5e_elbow_joint">
+            <joint name="ur5e_409_elbow_joint">
                 <command_interface name="position"/>
                 <command_interface name="velocity"/>
+                <command_interface name="effort"/>
                 <state_interface name="position">
-                  <param name="initial_value">${initial_positions['ur5e_elbow_joint']}</param>
+                  <param name="initial_value">${initial_positions['ur5e_409_elbow_joint']}</param>
                 </state_interface>
                 <state_interface name="velocity"/>
+                <state_interface name="effort"/>
             </joint>
-            <joint name="ur5e_wrist_1_joint">
+            <joint name="ur5e_409_wrist_1_joint">
                 <command_interface name="position"/>
                 <command_interface name="velocity"/>
+                <command_interface name="effort"/>
                 <state_interface name="position">
-                  <param name="initial_value">${initial_positions['ur5e_wrist_1_joint']}</param>
+                  <param name="initial_value">${initial_positions['ur5e_409_wrist_1_joint']}</param>
                 </state_interface>
                 <state_interface name="velocity"/>
+                <state_interface name="effort"/>
             </joint>
-            <joint name="ur5e_wrist_2_joint">
+            <joint name="ur5e_409_wrist_2_joint">
                 <command_interface name="position"/>
                 <command_interface name="velocity"/>
+                <command_interface name="effort"/>
                 <state_interface name="position">
-                  <param name="initial_value">${initial_positions['ur5e_wrist_2_joint']}</param>
+                  <param name="initial_value">${initial_positions['ur5e_409_wrist_2_joint']}</param>
                 </state_interface>
                 <state_interface name="velocity"/>
+                <state_interface name="effort"/>
             </joint>
-            <joint name="ur5e_wrist_3_joint">
+            <joint name="ur5e_409_wrist_3_joint">
                 <command_interface name="position"/>
                 <command_interface name="velocity"/>
+                <command_interface name="effort"/>
                 <state_interface name="position">
-                  <param name="initial_value">${initial_positions['ur5e_wrist_3_joint']}</param>
+                  <param name="initial_value">${initial_positions['ur5e_409_wrist_3_joint']}</param>
                 </state_interface>
                 <state_interface name="velocity"/>
+                <state_interface name="effort"/>
             </joint>
         </ros2_control>

File: src/Universal_Robots_ROS2_Tutorials/my_robot_cell/my_robot_cell_description/urdf/my_robot_cell_macro.xacro (robot description, xacro)
@@ -21,26 +21,25 @@
       <origin rpy="0 0 0" xyz="0 0 0"/>
     </xacro:safety_wall>
-    <link name="robot_mount"/>
-    <joint name="base_to_robot_mount" type="fixed">
-      <parent link="robot_base_plate"/>
-      <child link="robot_mount"/>
+    <link name="robot_mount_409"/>
+    <joint name="base_to_robot_mount_409" type="fixed">
+      <parent link="robot_base_plate_409"/>
+      <child link="robot_mount_409"/>
       <origin xyz="0 0 0" rpy="0 0 ${pi}" />
     </joint>
     <!--This will create the specific robot-->
     <xacro:ur_robot
-      name="${ur_type}"
-      tf_prefix="${ur_type}_"
-      parent="robot_mount"
+      name="${ur_type}_409"
+      tf_prefix="${ur_type}_409_"
+      parent="robot_mount_409"
       joint_limits_parameters_file="${joint_limits_parameters_file}"
       kinematics_parameters_file="${kinematics_parameters_file}"
       physical_parameters_file="${physical_parameters_file}"
-      visual_parameters_file="${visual_parameters_file}"
-    >
+      visual_parameters_file="${visual_parameters_file}"    >
       <origin xyz="0 0 0" rpy="0 0 0" />
     </xacro:ur_robot>
-    <xacro:box parent="ur5e_tool0">
+    <xacro:box parent="${ur_type}_409_tool0">
       <origin xyz="0 0 0.1" rpy="0 0 0"/>
     </xacro:box>
-    <!--xacro:onrobot_2fg7_gripper prefix= "onrobot_2fg7_gripper" parent="ur5e_tool0">
+    <!--xacro:onrobot_2fg7_gripper prefix= "onrobot_2fg7_gripper" parent="${ur_type}_409_tool0">
       <origin yxz="0 0 0" rpy="0 4.71239 0"/>
     </xacro:onrobot_2fg7_gripper-->

File: src/Universal_Robots_ROS2_Tutorials/my_robot_cell/my_robot_cell_description/urdf/table.xacro (robot description, xacro)
@@ -31,10 +31,39 @@
       </inertial>
     </link>
-    <joint name="robot_base_plate_joint" type="fixed">
+    <joint name="robot_base_plate_409_joint" type="fixed">
       <parent link="table" />
-      <child link="robot_base_plate"/>
+      <child link="robot_base_plate_409"/>
       <origin rpy="0 0 0" xyz="-0.52 0.32 0.02"/>
     </joint>
-    <link name="robot_base_plate">
+    <link name="robot_base_plate_409">
+      <visual>
+        <geometry>
+          <box size="0.16 0.16 0.02"/>
+        </geometry>
+        <origin xyz= "0 0 -0.01"/>
+        <material name="grey">
+          <color rgba="0.5 0.5 0.5 1.0"/>
+        </material>
+      </visual>
+      <collision>
+        <geometry>
+          <box size="0.16 0.16 0.01999"/>
+        </geometry>
+        <origin xyz= "0 0 -0.01"/>
+      </collision>
+      <inertial>
+        <mass value="2.0"/>
+        <inertia
+        ixx="1.0" ixy="0.0" ixz="0.0"
+        iyy="1.0" iyz="0.0"
+        izz="1.0"/>
+      </inertial>
+    </link>
+     <joint name="robot_base_plate_410_joint" type="fixed">
+      <parent link="table" />
+      <child link="robot_base_plate_410"/>
+      <origin rpy="0 0 0" xyz="0.52 -0.32 0.02"/>
+    </joint>
+    <link name="robot_base_plate_410">
       <visual>
         <geometry>

Commit message: All in urdf.xacro

File: src/Universal_Robots_ROS2_Tutorials/my_robot_cell/moveit_config/config/my_robot_cell.ros2_control.xacro (robot description, xacro)
@@ -8,63 +8,51 @@
                 <plugin>mock_components/GenericSystem</plugin>
             </hardware>
-            <joint name="ur5e_409_shoulder_pan_joint">
+            <joint name="ur5e_shoulder_pan_joint">
                 <command_interface name="position"/>
                 <command_interface name="velocity"/>
-                <command_interface name="effort"/>
                 <state_interface name="position">
-                  <param name="initial_value">${initial_positions['ur5e_409_shoulder_pan_joint']}</param>
+                  <param name="initial_value">${initial_positions['ur5e_shoulder_pan_joint']}</param>
                 </state_interface>
                 <state_interface name="velocity"/>
-                <state_interface name="effort"/>
             </joint>
-            <joint name="ur5e_409_shoulder_lift_joint">
+            <joint name="ur5e_shoulder_lift_joint">
                 <command_interface name="position"/>
                 <command_interface name="velocity"/>
-                <command_interface name="effort"/>
                 <state_interface name="position">
-                  <param name="initial_value">${initial_positions['ur5e_409_shoulder_lift_joint']}</param>
+                  <param name="initial_value">${initial_positions['ur5e_shoulder_lift_joint']}</param>
                 </state_interface>
                 <state_interface name="velocity"/>
-                <state_interface name="effort"/>
             </joint>
-            <joint name="ur5e_409_elbow_joint">
+            <joint name="ur5e_elbow_joint">
                 <command_interface name="position"/>
                 <command_interface name="velocity"/>
-                <command_interface name="effort"/>
                 <state_interface name="position">
-                  <param name="initial_value">${initial_positions['ur5e_409_elbow_joint']}</param>
+                  <param name="initial_value">${initial_positions['ur5e_elbow_joint']}</param>
                 </state_interface>
                 <state_interface name="velocity"/>
-                <state_interface name="effort"/>
             </joint>
-            <joint name="ur5e_409_wrist_1_joint">
+            <joint name="ur5e_wrist_1_joint">
                 <command_interface name="position"/>
                 <command_interface name="velocity"/>
-                <command_interface name="effort"/>
                 <state_interface name="position">
-                  <param name="initial_value">${initial_positions['ur5e_409_wrist_1_joint']}</param>
+                  <param name="initial_value">${initial_positions['ur5e_wrist_1_joint']}</param>
                 </state_interface>
                 <state_interface name="velocity"/>
-                <state_interface name="effort"/>
             </joint>
-            <joint name="ur5e_409_wrist_2_joint">
+            <joint name="ur5e_wrist_2_joint">
                 <command_interface name="position"/>
                 <command_interface name="velocity"/>
-                <command_interface name="effort"/>
                 <state_interface name="position">
-                  <param name="initial_value">${initial_positions['ur5e_409_wrist_2_joint']}</param>
+                  <param name="initial_value">${initial_positions['ur5e_wrist_2_joint']}</param>
                 </state_interface>
                 <state_interface name="velocity"/>
-                <state_interface name="effort"/>
             </joint>
-            <joint name="ur5e_409_wrist_3_joint">
+            <joint name="ur5e_wrist_3_joint">
                 <command_interface name="position"/>
                 <command_interface name="velocity"/>
-                <command_interface name="effort"/>
                 <state_interface name="position">
-                  <param name="initial_value">${initial_positions['ur5e_409_wrist_3_joint']}</param>
+                  <param name="initial_value">${initial_positions['ur5e_wrist_3_joint']}</param>
                 </state_interface>
                 <state_interface name="velocity"/>
-                <state_interface name="effort"/>
             </joint>
         </ros2_control>

File: src/Universal_Robots_ROS2_Tutorials/my_robot_cell/my_robot_cell_control/urdf/my_robot_cell_controlled.urdf.xacro (robot description, xacro)
@@ -5,4 +5,6 @@
   <!--The driver already provides a control tag for the UR arm, we can directly include-->
   <xacro:include filename="$(find ur_robot_driver)/urdf/ur.ros2_control.xacro"/>
+  <xacro:include filename="$(find my_robot_cell_description)/urdf/table.xacro"/>
+  <xacro:include filename="$(find my_robot_cell_description)/urdf/safety_wall.xacro"/>
   <!--We need to specify the arguments used for parametrizing our description-->
   <xacro:arg name="ur_type" default="ur5e"/>
@@ -19,4 +21,10 @@
   <xacro:arg name="mock_sensor_commands" default="false" />
   <link name="world" />
+  <xacro:table parent="world">
+    <origin rpy="0 0 0" xyz="0 -0 0.9"/>
+  </xacro:table>
+  <xacro:safety_wall parent="world">
+    <origin rpy="0 0 0" xyz="0 0 0"/>
+  </xacro:safety_wall>
   <!--Create the scene description including the robot-->
   <xacro:my_robot_cell
@@ -33,5 +41,5 @@
   <xacro:ur_ros2_control
     name="$(arg ur_type)"
-    tf_prefix="ur5e_409_"
+    tf_prefix="$(arg ur_type)_"
     kinematics_parameters_file="$(arg kinematics_parameters_file)"
     robot_ip="$(arg robot_ip)"

File: src/Universal_Robots_ROS2_Tutorials/my_robot_cell/my_robot_cell_description/urdf/my_robot_cell.urdf.xacro (robot description, xacro)
@@ -2,4 +2,6 @@
 <robot name="my_robot_cell" xmlns:xacro="http://ros.org/wiki/xacro">
   <xacro:include filename="$(find my_robot_cell_description)/urdf/my_robot_cell_macro.xacro"/>
+  <xacro:include filename="$(find my_robot_cell_description)/urdf/table.xacro"/>
+  <xacro:include filename="$(find my_robot_cell_description)/urdf/safety_wall.xacro"/>
   <xacro:arg name="ur_type" default="ur5e"/>
   <xacro:arg name="joint_limits_parameters_file" default="$(find ur_description)/config/$(arg ur_type)/joint_limits.yaml"/>
@@ -9,4 +11,10 @@
   <link name="world"/>
   <!--This will create the scene where the robot is located in-->
+  <xacro:table parent="world">
+    <origin rpy="0 0 0" xyz="0 -0 0.9"/>
+  </xacro:table>
+  <xacro:safety_wall parent="world">
+    <origin rpy="0 0 0" xyz="0 0 0"/>
+  </xacro:safety_wall>
   <xacro:my_robot_cell
     parent="world"

File: src/Universal_Robots_ROS2_Tutorials/my_robot_cell/my_robot_cell_description/urdf/my_robot_cell_macro.xacro (robot description, xacro)
@@ -2,6 +2,4 @@
 <robot xmlns:xacro="http://ros.org/wiki/xacro">
   <xacro:include filename="$(find ur_description)/urdf/ur_macro.xacro"/>
-  <xacro:include filename="$(find my_robot_cell_description)/urdf/safety_wall.xacro"/>
-  <xacro:include filename="$(find my_robot_cell_description)/urdf/table.xacro"/>
   <xacro:include filename="$(find my_robot_cell_description)/urdf/box.xacro"/>
   <xacro:include filename="$(find my_robot_cell_description)/urdf/2fg7_gripper/urdf/onrobot_2fg7_gripper.urdf.xacro"/>
@@ -15,31 +13,26 @@
     visual_parameters_file
     ">
-    <xacro:table parent="${parent}">
-      <origin rpy="0 0 0" xyz="0 -0 0.9"/>
-    </xacro:table>
-    <xacro:safety_wall parent="${parent}">
-      <origin rpy="0 0 0" xyz="0 0 0"/>
-    </xacro:safety_wall>
-    <link name="robot_mount_409"/>
-    <joint name="base_to_robot_mount_409" type="fixed">
-      <parent link="robot_base_plate_409"/>
-      <child link="robot_mount_409"/>
+    <link name="robot_mount"/>
+    <joint name="base_to_robot_mount" type="fixed">
+      <parent link="robot_base_plate"/>
+      <child link="robot_mount"/>
       <origin xyz="0 0 0" rpy="0 0 ${pi}" />
     </joint>
     <!--This will create the specific robot-->
     <xacro:ur_robot
-      name="${ur_type}_409"
-      tf_prefix="${ur_type}_409_"
-      parent="robot_mount_409"
+      name="${ur_type}"
+      tf_prefix="${ur_type}_"
+      parent="robot_mount"
       joint_limits_parameters_file="${joint_limits_parameters_file}"
       kinematics_parameters_file="${kinematics_parameters_file}"
       physical_parameters_file="${physical_parameters_file}"
-      visual_parameters_file="${visual_parameters_file}"    >
+      visual_parameters_file="${visual_parameters_file}"
+    >
       <origin xyz="0 0 0" rpy="0 0 0" />
     </xacro:ur_robot>
-    <xacro:box parent="${ur_type}_409_tool0">
+    <xacro:box parent="ur5e_tool0">
       <origin xyz="0 0 0.1" rpy="0 0 0"/>
     </xacro:box>
-    <!--xacro:onrobot_2fg7_gripper prefix= "onrobot_2fg7_gripper" parent="${ur_type}_409_tool0">
+    <!--xacro:onrobot_2fg7_gripper prefix= "onrobot_2fg7_gripper" parent="ur5e_tool0">
       <origin yxz="0 0 0" rpy="0 4.71239 0"/>
     </xacro:onrobot_2fg7_gripper-->

File: src/Universal_Robots_ROS2_Tutorials/my_robot_cell/my_robot_cell_description/urdf/table.xacro (robot description, xacro)
@@ -31,39 +31,10 @@
       </inertial>
     </link>
-    <joint name="robot_base_plate_409_joint" type="fixed">
+    <joint name="robot_base_plate_joint" type="fixed">
       <parent link="table" />
-      <child link="robot_base_plate_409"/>
+      <child link="robot_base_plate"/>
       <origin rpy="0 0 0" xyz="-0.52 0.32 0.02"/>
     </joint>
-    <link name="robot_base_plate_409">
-      <visual>
-        <geometry>
-          <box size="0.16 0.16 0.02"/>
-        </geometry>
-        <origin xyz= "0 0 -0.01"/>
-        <material name="grey">
-          <color rgba="0.5 0.5 0.5 1.0"/>
-        </material>
-      </visual>
-      <collision>
-        <geometry>
-          <box size="0.16 0.16 0.01999"/>
-        </geometry>
-        <origin xyz= "0 0 -0.01"/>
-      </collision>
-      <inertial>
-        <mass value="2.0"/>
-        <inertia
-        ixx="1.0" ixy="0.0" ixz="0.0"
-        iyy="1.0" iyz="0.0"
-        izz="1.0"/>
-      </inertial>
-    </link>
-     <joint name="robot_base_plate_410_joint" type="fixed">
-      <parent link="table" />
-      <child link="robot_base_plate_410"/>
-      <origin rpy="0 0 0" xyz="0.52 -0.32 0.02"/>
-    </joint>
-    <link name="robot_base_plate_410">
+    <link name="robot_base_plate">
       <visual>
         <geometry>
