Commit message: parametrized first arm

File: src/Universal_Robots_ROS2_Tutorials/my_robot_cell/my_robot_cell_control/urdf/my_robot_cell_controlled.urdf.xacro (robot description, xacro)
@@ -29,4 +29,5 @@
   <!--Create the scene description including the robot-->
   <xacro:my_robot_cell
+    prefix="409_"
     parent="world"
     ur_type="$(arg ur_type)"
@@ -41,5 +42,5 @@
   <xacro:ur_ros2_control
     name="$(arg ur_type)"
-    tf_prefix="$(arg ur_type)_"
+    tf_prefix="409_$(arg ur_type)_"
     kinematics_parameters_file="$(arg kinematics_parameters_file)"
     robot_ip="$(arg robot_ip)"

File: src/Universal_Robots_ROS2_Tutorials/my_robot_cell/my_robot_cell_description/urdf/box.xacro (robot description, xacro)
@@ -2,10 +2,10 @@
 <robot xmlns:xacro="http://ros.org/wiki/xacro">
   <xacro:macro name="box" params="parent *origin">
-    <joint name="box_joint" type="fixed">
-      <parent link="ur5e_tool0" />
-      <child link="box" />
+    <joint name="${prefix}box_joint" type="fixed">
+      <parent link="${prefix}ur5e_tool0" />
+      <child link="${prefix}box" />
       <origin rpy="0 0 0" xyz="0 0 0.16"/>
     </joint>
-    <link name="box">
+    <link name="${prefix}box">
       <visual>
         <geometry>

File: src/Universal_Robots_ROS2_Tutorials/my_robot_cell/my_robot_cell_description/urdf/my_robot_cell.urdf.xacro (robot description, xacro)
@@ -19,4 +19,5 @@
   <xacro:my_robot_cell
     parent="world"
+    prefix="409_"
     ur_type="$(arg ur_type)"
     joint_limits_parameters_file="$(arg joint_limits_parameters_file)"

File: src/Universal_Robots_ROS2_Tutorials/my_robot_cell/my_robot_cell_description/urdf/my_robot_cell_macro.xacro (robot description, xacro)
@@ -7,4 +7,5 @@
     parent
     *origin
+    prefix
     ur_type
     joint_limits_parameters_file
@@ -13,15 +14,15 @@
     visual_parameters_file
     ">
-    <link name="robot_mount"/>
-    <joint name="base_to_robot_mount" type="fixed">
-      <parent link="robot_base_plate"/>
-      <child link="robot_mount"/>
+    <link name="${prefix}robot_mount"/>
+    <joint name="${prefix}base_to_robot_mount" type="fixed">
+      <parent link="${prefix}robot_base_plate"/>
+      <child link="${prefix}robot_mount"/>
       <origin xyz="0 0 0" rpy="0 0 ${pi}" />
     </joint>
     <!--This will create the specific robot-->
     <xacro:ur_robot
-      name="${ur_type}"
-      tf_prefix="${ur_type}_"
-      parent="robot_mount"
+      name="${prefix}${ur_type}"
+      tf_prefix="${prefix}${ur_type}_"
+      parent="${prefix}robot_mount"
       joint_limits_parameters_file="${joint_limits_parameters_file}"
       kinematics_parameters_file="${kinematics_parameters_file}"
@@ -31,5 +32,5 @@
       <origin xyz="0 0 0" rpy="0 0 0" />
     </xacro:ur_robot>
-    <xacro:box parent="ur5e_tool0">
+    <xacro:box parent="${prefix}ur5e_tool0">
       <origin xyz="0 0 0.1" rpy="0 0 0"/>
     </xacro:box>

File: src/Universal_Robots_ROS2_Tutorials/my_robot_cell/my_robot_cell_description/urdf/table.xacro (robot description, xacro)
@@ -3,5 +3,5 @@
   <xacro:macro name="table" params="parent *origin">
     <joint name="table_base_joint" type="fixed">
-      <parent link="${parent}" />
+      <parent link="world" />
       <child link="table" />
       <origin rpy="0 0 0" xyz="0 0 0.9"/>
@@ -31,10 +31,10 @@
       </inertial>
     </link>
-    <joint name="robot_base_plate_joint" type="fixed">
+    <joint name="409_robot_base_plate_joint" type="fixed">
       <parent link="table" />
-      <child link="robot_base_plate"/>
+      <child link="409_robot_base_plate"/>
       <origin rpy="0 0 0" xyz="-0.52 0.32 0.02"/>
     </joint>
-    <link name="robot_base_plate">
+    <link name="409_robot_base_plate">
       <visual>
         <geometry>

Commit message: finally trying to integrate two robots

File: src/Universal_Robots_ROS2_Tutorials/my_robot_cell/my_robot_cell_control/urdf/my_robot_cell_controlled.urdf.xacro (robot description, xacro)
@@ -41,5 +41,5 @@
   <!--Create the control tag for the UR robot-->
   <xacro:ur_ros2_control
-    name="$(arg ur_type)"
+    name="409_ur5e"
     tf_prefix="409_$(arg ur_type)_"
     kinematics_parameters_file="$(arg kinematics_parameters_file)"
@@ -52,4 +52,28 @@
     headless_mode="$(arg headless_mode)"
   />
+  <xacro:my_robot_cell
+    prefix="410_"
+    parent="world"
+    ur_type="$(arg ur_type)"
+    joint_limits_parameters_file="$(arg joint_limit_parameters_file)"
+    kinematics_parameters_file="$(arg kinematics_parameters_file)"
+    physical_parameters_file="$(arg physical_parameters_file)"
+    visual_parameters_file="$(arg visual_parameters_file)"
+>
+    <!-- Change position so it's not overlapping with first robot -->
+    <origin xyz="0 0 1" rpy="0 0 0" />
+</xacro:my_robot_cell>
+  <xacro:ur_ros2_control
+    name="410_ur5e"
+    tf_prefix="410_$(arg ur_type)_"
+    kinematics_parameters_file="$(arg kinematics_parameters_file)"
+    robot_ip="192.168.1.103"
+    script_filename="$(arg ur_script_filename)"
+    output_recipe_filename="$(arg ur_output_recipe_filename)"
+    input_recipe_filename="$(arg ur_input_recipe_filename)"
+    use_mock_hardware="$(arg use_mock_hardware)"
+    mock_sensor_commands="$(arg mock_sensor_commands)"
+    headless_mode="$(arg headless_mode)"
+  />
   <!--If you had more controlled devices in your description, e.g. a gripper, you can add another ros2_control tag here-->
 </robot>

File: src/Universal_Robots_ROS2_Tutorials/my_robot_cell/my_robot_cell_description/urdf/my_robot_cell.urdf.xacro (robot description, xacro)
@@ -28,3 +28,14 @@
       <origin xyz="0 0 0" rpy="0 0 0" />
   </xacro:my_robot_cell>
+  <xacro:my_robot_cell
+    parent="world"
+    prefix="410_"
+    ur_type="$(arg ur_type)"
+    joint_limits_parameters_file="$(arg joint_limits_parameters_file)"
+    kinematics_parameters_file="$(arg kinematics_parameters_file)"
+    physical_parameters_file="$(arg physical_parameters_file)"
+    visual_parameters_file="$(arg visual_parameters_file)"
+    >
+      <origin xyz="0 0 0" rpy="0 0 0" />
+  </xacro:my_robot_cell>
 </robot>

File: src/Universal_Robots_ROS2_Tutorials/my_robot_cell/my_robot_cell_description/urdf/table.xacro (robot description, xacro)
@@ -60,4 +60,33 @@
       </inertial>
     </link>
+    <joint name="410_robot_base_plate_joint" type="fixed">
+      <parent link="table" />
+      <child link="410_robot_base_plate"/>
+      <origin rpy="0 0 0" xyz="0.52 -0.32 0.02"/>
+    </joint>
+    <link name="410_robot_base_plate">
+      <visual>
+        <geometry>
+          <box size="0.16 0.16 0.02"/>
+        </geometry>
+        <origin xyz= "0 0 -0.01"/>
+        <material name="grey">
+          <color rgba="0.5 0.5 0.5 1.0"/>
+        </material>
+      </visual>
+      <collision>
+        <geometry>
+          <box size="0.16 0.16 0.01999"/>
+        </geometry>
+        <origin xyz= "0 0 -0.01"/>
+      </collision>
+      <inertial>
+        <mass value="2.0"/>
+        <inertia
+        ixx="1.0" ixy="0.0" ixz="0.0"
+        iyy="1.0" iyz="0.0"
+        izz="1.0"/>
+      </inertial>
+    </link>
   </xacro:macro>
 </robot>

Commit message: dual arm motion planning working. no refined coordinates

File: src/Universal_Robots_ROS2_Tutorials/my_robot_cell/my_robot_cell_control/urdf/my_robot_cell_controlled.urdf.xacro (robot description, xacro)
@@ -30,4 +30,5 @@
   <!--Create the scene description including the robot-->
   <xacro:my_robot_cell
+    rotation="0 0 0"
     prefix="409_"
     parent="world"
@@ -58,4 +59,5 @@
   />
   <xacro:my_robot_cell
+    rotation="0 0 -${pi/2}"
     prefix="410_"
     parent="world"

File: src/Universal_Robots_ROS2_Tutorials/my_robot_cell/my_robot_cell_description/urdf/my_robot_cell.urdf.xacro (robot description, xacro)
@@ -18,4 +18,5 @@
   </xacro:safety_wall>
   <xacro:my_robot_cell
+    rotation="0 0 0"
     parent="world"
     prefix="409_"
@@ -29,4 +30,5 @@
   </xacro:my_robot_cell>
   <xacro:my_robot_cell
+    rotation="0 0  -${pi/2}"
     parent="world"
     prefix="410_"

File: src/Universal_Robots_ROS2_Tutorials/my_robot_cell/my_robot_cell_description/urdf/my_robot_cell_macro.xacro (robot description, xacro)
@@ -6,4 +6,5 @@
   <xacro:macro name="my_robot_cell" params="
     parent
+    rotation
     *origin
     prefix
@@ -30,5 +31,5 @@
       visual_parameters_file="${visual_parameters_file}"
     >
-      <origin xyz="0 0 0" rpy="0 0 0" />
+      <origin xyz="0 0 0" rpy="${rotation}" />
     </xacro:ur_robot>
     <xacro:box parent="${prefix}ur5e_tool0">
